File: Robots/Weeder/Chassis/HW/CL_Mot_Drv_Enc_Ard_Shield/CL_Mot_Drv_Enc_Ard_Shield.kicad_sch (KiCad schematic)
At the start: 4 parts

Commit message: Soldering PCB.
Parts:
- added H1, H2, H3, H4: MountingHole, MountingHole:MountingHole_3mm, symbol Mechanical:MountingHole
- added J3: Screw_Terminal_01x04, TerminalBlock:TerminalBlock_bornier-4_P5.08mm, symbol Connector:Screw_Terminal_01x04
- CON1: renamed from CON?; footprint (none) -> Connector_IDC:IDC-Header_2x10_P2.54mm_Vertical
- J1, J2: renamed from J?; value Conn_01x05 -> 1x5 2.54mm female; footprint (none) -> Connector_PinSocket_2.54mm:PinSocket_1x05_P2.54mm_Vertical
- gave numbers to parts that had none: 1
Connections:
- net GND: now also A1.7 (GND), J3.2 (Pin_2)
- net UH: now also A1.28 (D13); no longer A1.23 (D8)
- net UL: now also A1.27 (D12); no longer A1.24 (D9)
- net VH: now also A1.26 (D11); no longer A1.25 (D10)
- net VL: now also A1.25 (D10); no longer A1.26 (D11)
- net WH: now also A1.24 (D9); no longer A1.27 (D12)
- net WL: now also A1.23 (D8); no longer A1.28 (D13)
- net U_SSD_L: now reaches A1.17 (D2)
- net U_SSD_H: now reaches A1.18 (D3)
- net V_SSD_L: now reaches A1.19 (D4)
- net V_SSD_H: now reaches A1.20 (D5)
- new net +24V: J3.1 (Pin_1)
- new net U_COLD: J3.3 (Pin_3)
- new net V_COLD: J3.4 (Pin_4)
Other:
- added sheet ssr_u (SSR.kicad_sch)
- added sheet ssr_v (SSR.kicad_sch)
- note added: "TODO Swap in SW"
- note removed: "TODO Nch IRFL to src to GND"
- note removed: "TODO Swap here and in SW"
