File: Industrial/AC_Logger/HW/AFE/Amp.kicad_sch (KiCad schematic)
At the start: 10 parts, among them U1 TL072

Commit message: Some error recovery.
Parts:
- renumbered C2 to C?, D1 to D?, D3 to D?, D4 to D?, D2 to D?, R8 to R?, R7 to R?, R9 to R?, R6 to R?, U1 to U?
Changed lines of the file:
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@@
   (symbol (lib_id "power:VEE") (at 78.74 48.26 180) (unit 1)
     (in_bom yes) (on_board yes)
-    (property "Reference" "#PWR023" (id 0) (at 78.74 44.45 0)
+    (property "Reference" "#PWR?" (id 0) (at 78.74 44.45 0)
       (effects (font (size 1.27 1.27)) hide)
     )
@@
   (symbol (lib_id "power:VCC") (at 78.74 27.94 0) (unit 1)
     (in_bom yes) (on_board yes)
-    (property "Reference" "#PWR022" (id 0) (at 78.74 31.75 0)
+    (property "Reference" "#PWR?" (id 0) (at 78.74 31.75 0)
       (effects (font (size 1.27 1.27)) hide)
     )
@@
   (symbol (lib_id "Device:C") (at 66.04 38.1 0) (unit 1)
     (in_bom yes) (on_board yes)
-    (property "Reference" "C2" (id 0) (at 68.961 36.9316 0)
+    (property "Reference" "C?" (id 0) (at 68.961 36.9316 0)
       (effects (font (size 1.27 1.27)) (justify left))
     )
@@
   (symbol (lib_id "Amplifier_Operational:TL072") (at 114.3 68.58 0) (unit 1)
     (in_bom yes) (on_board yes)
-    (property "Reference" "U1" (id 0) (at 114.3 59.2582 0))
+    (property "Reference" "U?" (id 0) (at 114.3 59.2582 0))
     (property "Value" "TL072" (id 1) (at 114.3 61.5696 0))
     (property "Footprint" "Package_DIP:DIP-8_W7.62mm" (id 2) (at 114.3 68.58 0)
@@
   (symbol (lib_id "Amplifier_Operational:TL072") (at 113.03 101.6 0) (unit 2)
     (in_bom yes) (on_board yes)
-    (property "Reference" "U1" (id 0) (at 113.03 92.2782 0))
+    (property "Reference" "U?" (id 0) (at 113.03 92.2782 0))
     (property "Value" "TL072" (id 1) (at 113.03 94.5896 0))
     (property "Footprint" "Package_DIP:DIP-8_W7.62mm" (id 2) (at 113.03 101.6 0)
@@
   (symbol (lib_id "Amplifier_Operational:TL072") (at 81.28 38.1 0) (unit 3)
     (in_bom yes) (on_board yes)
-    (property "Reference" "U1" (id 0) (at 80.2132 36.9316 0)
+    (property "Reference" "U?" (id 0) (at 80.2132 36.9316 0)
       (effects (font (size 1.27 1.27)) (justify left))
     )
@@
   (symbol (lib_id "power:VDDF") (at 104.14 58.42 0) (unit 1)
     (in_bom yes) (on_board yes)
-    (property "Reference" "#PWR024" (id 0) (at 104.14 62.23 0)
+    (property "Reference" "#PWR?" (id 0) (at 104.14 62.23 0)
       (effects (font (size 1.27 1.27)) hide)
     )
@@
   (symbol (lib_id "Device:R") (at 111.76 82.55 270) (unit 1)
     (in_bom yes) (on_board yes)
-    (property "Reference" "R8" (id 0) (at 111.76 77.2922 90))
+    (property "Reference" "R?" (id 0) (at 111.76 77.2922 90))
     (property "Value" "220k" (id 1) (at 111.76 79.6036 90))
     (property "Footprint" "Resistor_THT:R_Axial_DIN0207_L6.3mm_D2.5mm_P2.54mm_Vertical" (id 2) (at 111.76 80.772 90)
@@
   (symbol (lib_id "Device:R") (at 101.6 71.12 270) (unit 1)
     (in_bom yes) (on_board yes)
-    (property "Reference" "R7" (id 0) (at 101.6 65.8622 90))
+    (property "Reference" "R?" (id 0) (at 101.6 65.8622 90))
     (property "Value" "100k" (id 1) (at 101.6 68.1736 90))
     (property "Footprint" "For_Rasterboard:R_Axial_DIN0207_L6.3mm_D2.5mm_Pinf_Horizontal" (id 2) (at 101.6 69.342 90)
@@
   (symbol (lib_id "Device:R") (at 111.76 115.57 270) (unit 1)
     (in_bom yes) (on_board yes)
-    (property "Reference" "R9" (id 0) (at 111.76 110.3122 90))
+    (property "Reference" "R?" (id 0) (at 111.76 110.3122 90))
     (property "Value" "220k" (id 1) (at 111.76 112.6236 90))
     (property "Footprint" "Resistor_THT:R_Axial_DIN0207_L6.3mm_D2.5mm_P2.54mm_Vertical" (id 2) (at 111.76 113.792 90)
@@
   (symbol (lib_id "Device:R") (at 100.33 104.14 270) (unit 1)
     (in_bom yes) (on_board yes)
-    (property "Reference" "R6" (id 0) (at 100.33 98.8822 90))
+    (property "Reference" "R?" (id 0) (at 100.33 98.8822 90))
     (property "Value" "100k" (id 1) (at 100.33 101.1936 90))
     (property "Footprint" "For_Rasterboard:R_Axial_DIN0207_L6.3mm_D2.5mm_Pinf_Horizontal" (id 2) (at 100.33 102.362 90)
@@
   (symbol (lib_id "power:VDDF") (at 104.14 91.44 0) (unit 1)
     (in_bom yes) (on_board yes)
-    (property "Reference" "#PWR025" (id 0) (at 104.14 95.25 0)
+    (property "Reference" "#PWR?" (id 0) (at 104.14 95.25 0)
       (effects (font (size 1.27 1.27)) hide)
     )
@@
   (symbol (lib_id "Device:D_Filled") (at 66.04 74.93 270) (unit 1)
     (in_bom yes) (on_board yes)
-    (property "Reference" "D1" (id 0) (at 68.0466 73.7616 90)
+    (property "Reference" "D?" (id 0) (at 68.0466 73.7616 90)
       (effects (font (size 1.27 1.27)) (justify left))
     )
@@
   (symbol (lib_id "Device:D_Filled") (at 77.47 74.93 90) (unit 1)
     (in_bom yes) (on_board yes)
-    (property "Reference" "D3" (id 0) (at 79.4766 73.7616 90)
+    (property "Reference" "D?" (id 0) (at 79.4766 73.7616 90)
       (effects (font (size 1.27 1.27)) (justify right))
     )
@@
   (symbol (lib_id "Device:D_Filled") (at 77.47 107.95 90) (unit 1)
     (in_bom yes) (on_board yes)
-    (property "Reference" "D4" (id 0) (at 79.4766 106.7816 90)
+    (property "Reference" "D?" (id 0) (at 79.4766 106.7816 90)
       (effects (font (size 1.27 1.27)) (justify right))
     )
@@
   (symbol (lib_id "Device:D_Filled") (at 66.04 107.95 270) (unit 1)
     (in_bom yes) (on_board yes)
-    (property "Reference" "D2" (id 0) (at 68.0466 106.7816 90)
+    (property "Reference" "D?" (id 0) (at 68.0466 106.7816 90)
       (effects (font (size 1.27 1.27)) (justify left))
     )
@@
   (symbol (lib_id "power:GND") (at 77.47 114.3 0) (unit 1)
     (in_bom yes) (on_board yes)
-    (property "Reference" "#PWR021" (id 0) (at 77.47 120.65 0)
+    (property "Reference" "#PWR?" (id 0) (at 77.47 120.65 0)
       (effects (font (size 1.27 1.27)) hide)
     )
@@
   (symbol (lib_id "power:GND") (at 66.04 114.3 0) (unit 1)
     (in_bom yes) (on_board yes)
-    (property "Reference" "#PWR019" (id 0) (at 66.04 120.65 0)
+    (property "Reference" "#PWR?" (id 0) (at 66.04 120.65 0)
       (effects (font (size 1.27 1.27)) hide)
     )
@@
   (symbol (lib_id "power:GND") (at 66.04 81.28 0) (unit 1)
     (in_bom yes) (on_board yes)
-    (property "Reference" "#PWR018" (id 0) (at 66.04 87.63 0)
+    (property "Reference" "#PWR?" (id 0) (at 66.04 87.63 0)
       (effects (font (size 1.27 1.27)) hide)
     )
@@
   (symbol (lib_id "power:GND") (at 77.47 81.28 0) (unit 1)
     (in_bom yes) (on_board yes)
-    (property "Reference" "#PWR020" (id 0) (at 77.47 87.63 0)
-      (effects (font (size 1.27 1.27)) hide)
-    )
+    (property "Reference" "#PWR?" (id 0) (at 77.47 87.63 0)
+      (effects (font (size 1.27 1.27)) hide)
+    )
