File: Industrial/AC_Logger/HW/AFE/Sensor.kicad_sch (KiCad schematic)
At the start: 4 parts, among them T1 ASM-010

Commit message: Some error recovery.
Parts:
- renumbered R5 to R?, R4 to R?, R3 to R?, T1 to T?
Changed lines of the file:
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@@
   (symbol (lib_id "Device:Transformer_1P_1S") (at 93.98 74.93 270) (mirror x) (unit 1)
     (in_bom yes) (on_board yes)
-    (property "Reference" "T1" (id 0) (at 86.6902 76.0984 90)
+    (property "Reference" "T?" (id 0) (at 86.6902 76.0984 90)
       (effects (font (size 1.27 1.27)) (justify right))
     )
@@
   (symbol (lib_id "power:GND") (at 88.9 87.63 0) (unit 1)
     (in_bom yes) (on_board yes)
-    (property "Reference" "#PWR015" (id 0) (at 88.9 93.98 0)
+    (property "Reference" "#PWR?" (id 0) (at 88.9 93.98 0)
       (effects (font (size 1.27 1.27)) hide)
     )
@@
   (symbol (lib_id "power:GND") (at 109.22 102.87 0) (unit 1)
     (in_bom yes) (on_board yes)
-    (property "Reference" "#PWR016" (id 0) (at 109.22 109.22 0)
+    (property "Reference" "#PWR?" (id 0) (at 109.22 109.22 0)
       (effects (font (size 1.27 1.27)) hide)
     )
@@
   (symbol (lib_id "power:GND") (at 127 85.09 0) (unit 1)
     (in_bom yes) (on_board yes)
-    (property "Reference" "#PWR017" (id 0) (at 127 91.44 0)
+    (property "Reference" "#PWR?" (id 0) (at 127 91.44 0)
       (effects (font (size 1.27 1.27)) hide)
     )
@@
   (symbol (lib_id "Device:R") (at 127 80.01 0) (unit 1)
     (in_bom yes) (on_board yes)
-    (property "Reference" "R5" (id 0) (at 128.778 78.8416 0)
+    (property "Reference" "R?" (id 0) (at 128.778 78.8416 0)
       (effects (font (size 1.27 1.27)) (justify left))
     )
@@
   (symbol (lib_id "Device:R") (at 127 68.58 0) (unit 1)
     (in_bom yes) (on_board yes)
-    (property "Reference" "R4" (id 0) (at 128.778 67.4116 0)
+    (property "Reference" "R?" (id 0) (at 128.778 67.4116 0)
       (effects (font (size 1.27 1.27)) (justify left))
     )
@@
   (symbol (lib_id "Device:R") (at 109.22 97.79 0) (unit 1)
     (in_bom yes) (on_board yes)
-    (property "Reference" "R3" (id 0) (at 110.998 96.6216 0)
+    (property "Reference" "R?" (id 0) (at 110.998 96.6216 0)
       (effects (font (size 1.27 1.27)) (justify left))
     )
