File: Industrial/AC_Logger/HW/AFE/AFE.kicad_sch (KiCad schematic)
At the start: 3 parts

Commit message: Corrections.
Changed lines of the file:
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@@
     (effects (font (size 1.27 1.27)) (justify left bottom))
   )
-  (hierarchical_label "E1_OR_S3_OUT" (shape output) (at 146.05 90.17 0)
+  (hierarchical_label "S3_OUT" (shape output) (at 146.05 90.17 0)
     (effects (font (size 1.27 1.27)) (justify left))
   )
@@
     (effects (font (size 1.27 1.27)) (justify left))
   )
-  (hierarchical_label "E1_OR_S3_IN" (shape input) (at 57.15 90.17 180)
+  (hierarchical_label "S3_IN" (shape input) (at 57.15 90.17 180)
     (effects (font (size 1.27 1.27)) (justify right))
   )
