File: Industrial/AC_Logger/HW/Box/Box.kicad_sch (KiCad schematic)
At the start: 7 parts, among them J1 IEC C14 male socket, J2 IEC C14 male socket, J3 3ph AC socket, J4 1ph AC schuko socket, K1 FINDER-55.32.8.230.0040, K2 FINDER-55.32.8.230.0040

Commit message: Corrections.
Connections:
- net L1_IN is gone; now on net L1_OR_R3_IN: J1.1 (Pin_1), K1.24, K1.A1, K2.14
- net GND: now also J3.1 (Pin_1)
- net L1_OR_R3_IN: no longer K1.21, K2.21
- net L1_OR_R3__OUT: no longer names the net of J4.1 (Pin_1)
- net L1_OR_R3__OUT: no longer J3.1 (Pin_1)
- net R3_IN: no longer names the net of J2.1 (Pin_1)
- net R3_IN: no longer K1.22
- new net L1_OR_R3: K1.21, K2.21
- no-connect marks 3 -> 5
Other:
- sheet AFE ports: added S3_IN, S3_OUT; removed E1_OR_S3_IN, E1_OR_S3_OUT
- note removed: "If 3φ pluged, then L1_IN is off, then R3 is passed."
- moved on the sheet: J1, J2

Commit message: Corrected relay sym.
Parts:
- K1, K2: footprint (none) -> Relay_THT:Relay_DPDT_Finder_40.52
Connections:
- net L1_OR_R3: now also K1.41, K2.41; no longer K1.21, K2.21
- net L1_OR_R3_IN: now also K1.44; no longer K1.24
- net N_IN: now also K2.44; no longer K2.24

Commit message: Refactoring.
Parts:
- removed K1, K2: FINDER-55.32.8.230.0040, Relay_THT:Relay_DPDT_Finder_40.52, symbol Local_Relays:FINDER-55.32.8.230.0040
- removed LA?: FINDER-99.02.0.230.98, symbol Device:Lamp
Connections:
- no-connect marks 5 -> 1
Other:
- added sheet unnulling (Unnulling.kicad_sch)
- note removed: "Alway have ~7mA to E but that is below FID"
- note removed: "Correct"
- note removed: "Wrong"

Commit message: New brd.
Other:
- removed sheet unnulling
- added sheet unnulling1 (../Unnulling/Unnulling.kicad_sch)
