File: Industrial/AC_Logger/HW/PSU/PSU.kicad_sch (KiCad schematic)
At the start: 15 parts, among them U1 L7809, U2 L7909

Commit message: Some error recovery.
Parts:
- T?: footprint (none) -> For_Rasterboard:Transformer-3VA_2xSec
Changed lines of the file:
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@@
     (property "Reference" "T?" (id 0) (at 85.09 45.72 0))
     (property "Value" "230V 3.2VA - 2x 12V 1.6VA" (id 1) (at 85.09 48.26 0))
-    (property "Footprint" "" (id 2) (at 85.09 60.96 0)
+    (property "Footprint" "For_Rasterboard:Transformer-3VA_2xSec" (id 2) (at 85.09 60.96 0)
       (effects (font (size 1.27 1.27)) hide)
     )

Commit message: New brd.
Parts:
- removed H1, H2, H3, H4: MountingHole, MountingHole:MountingHole_3.2mm_M3_ISO7380_Pad, symbol Mechanical:MountingHole
- gave numbers to parts that had none: 1
Changed lines of the file:
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@@
     (effects (font (size 1.27 1.27)) (justify right))
-  )
-  (symbol (lib_id "Mechanical:MountingHole") (at 252.73 36.83 0) (unit 1)
-    (in_bom yes) (on_board yes)
-    (property "Reference" "H4" (id 0) (at 255.27 35.6616 0)
-      (effects (font (size 1.27 1.27)) (justify left))
-    )
-    (property "Value" "MountingHole" (id 1) (at 255.27 37.973 0)
-      (effects (font (size 1.27 1.27)) (justify left))
-    )
-    (property "Footprint" "MountingHole:MountingHole_3.2mm_M3_ISO7380_Pad" (id 2) (at 252.73 36.83 0)
-      (effects (font (size 1.27 1.27)) hide)
-    )
-    (property "Datasheet" "~" (id 3) (at 252.73 36.83 0)
-      (effects (font (size 1.27 1.27)) hide)
-    )
   )
   (symbol (lib_id "Device:Fuse") (at 107.95 71.12 90) (unit 1)
@@
   (symbol (lib_id "Device:Transformer_1P_2S") (at 85.09 60.96 0) (unit 1)
     (in_bom yes) (on_board yes) (fields_autoplaced)
-    (property "Reference" "T?" (id 0) (at 85.09 45.72 0))
+    (property "Reference" "T1" (id 0) (at 85.09 45.72 0))
     (property "Value" "230V 3.2VA - 2x 12V 1.6VA" (id 1) (at 85.09 48.26 0))
     (property "Footprint" "For_Rasterboard:Transformer-3VA_2xSec" (id 2) (at 85.09 60.96 0)
@@
     (pin "2")
   )
-  (symbol (lib_id "Mechanical:MountingHole") (at 38.1 27.94 0) (unit 1)
-    (in_bom yes) (on_board yes)
-    (property "Reference" "H2" (id 0) (at 40.64 26.7716 0)
-      (effects (font (size 1.27 1.27)) (justify left))
-    )
-    (property "Value" "MountingHole" (id 1) (at 40.64 29.083 0)
-      (effects (font (size 1.27 1.27)) (justify left))
-    )
-    (property "Footprint" "MountingHole:MountingHole_3.2mm_M3_ISO7380_Pad" (id 2) (at 38.1 27.94 0)
-      (effects (font (size 1.27 1.27)) hide)
-    )
-    (property "Datasheet" "~" (id 3) (at 38.1 27.94 0)
-      (effects (font (size 1.27 1.27)) hide)
-    )
-  )
-  (symbol (lib_id "Mechanical:MountingHole") (at 34.29 130.81 0) (unit 1)
-    (in_bom yes) (on_board yes)
-    (property "Reference" "H1" (id 0) (at 36.83 129.6416 0)
-      (effects (font (size 1.27 1.27)) (justify left))
-    )
-    (property "Value" "MountingHole" (id 1) (at 36.83 131.953 0)
-      (effects (font (size 1.27 1.27)) (justify left))
-    )
-    (property "Footprint" "MountingHole:MountingHole_3.2mm_M3_ISO7380_Pad" (id 2) (at 34.29 130.81 0)
-      (effects (font (size 1.27 1.27)) hide)
-    )
-    (property "Datasheet" "~" (id 3) (at 34.29 130.81 0)
-      (effects (font (size 1.27 1.27)) hide)
-    )
-  )
   (symbol (lib_id "Device:C") (at 217.17 92.71 180) (unit 1)
     (in_bom yes) (on_board yes)
@@
     (pin "2")
   )
-  (symbol (lib_id "Mechanical:MountingHole") (at 248.92 133.35 0) (unit 1)
-    (in_bom yes) (on_board yes)
-    (property "Reference" "H3" (id 0) (at 251.46 132.1816 0)
-      (effects (font (size 1.27 1.27)) (justify left))
-    )
-    (property "Value" "MountingHole" (id 1) (at 251.46 134.493 0)
-      (effects (font (size 1.27 1.27)) (justify left))
-    )
-    (property "Footprint" "MountingHole:MountingHole_3.2mm_M3_ISO7380_Pad" (id 2) (at 248.92 133.35 0)
-      (effects (font (size 1.27 1.27)) hide)
-    )
-    (property "Datasheet" "~" (id 3) (at 248.92 133.35 0)
-      (effects (font (size 1.27 1.27)) hide)
-    )
-  )
   (symbol (lib_id "power:VCC") (at 231.14 60.96 270) (mirror x) (unit 1)
