File: Industrial/AC_Logger/HW/PSU_Board/PSU_Board.kicad_sch (KiCad schematic)
At the start: 2 parts, among them J1 Screw_Terminal_01x02, J2 NS25-W3P male

Commit message: New brd.
Parts:
- added H1, H2, H3, H4: MountingHole, MountingHole:MountingHole_3.2mm_M3_ISO7380_Pad, symbol Mechanical:MountingHole
Changed lines of the file:
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@@
     (stroke (width 0) (type default) (color 0 0 0 0))
+  )
+  (symbol (lib_id "Mechanical:MountingHole") (at 40.64 134.62 0) (unit 1)
+    (in_bom yes) (on_board yes)
+    (property "Reference" "H1" (id 0) (at 43.18 133.4516 0)
+      (effects (font (size 1.27 1.27)) (justify left))
+    )
+    (property "Value" "MountingHole" (id 1) (at 43.18 135.763 0)
+      (effects (font (size 1.27 1.27)) (justify left))
+    )
+    (property "Footprint" "MountingHole:MountingHole_3.2mm_M3_ISO7380_Pad" (id 2) (at 40.64 134.62 0)
+      (effects (font (size 1.27 1.27)) hide)
+    )
+    (property "Datasheet" "~" (id 3) (at 40.64 134.62 0)
+      (effects (font (size 1.27 1.27)) hide)
+    )
   )
   (symbol (lib_id "Connector:Screw_Terminal_01x02") (at 97.79 78.74 0) (mirror y) (unit 1)
@@
     (pin "3")
   )
+  (symbol (lib_id "Mechanical:MountingHole") (at 44.45 31.75 0) (unit 1)
+    (in_bom yes) (on_board yes)
+    (property "Reference" "H2" (id 0) (at 46.99 30.5816 0)
+      (effects (font (size 1.27 1.27)) (justify left))
+    )
+    (property "Value" "MountingHole" (id 1) (at 46.99 32.893 0)
+      (effects (font (size 1.27 1.27)) (justify left))
+    )
+    (property "Footprint" "MountingHole:MountingHole_3.2mm_M3_ISO7380_Pad" (id 2) (at 44.45 31.75 0)
+      (effects (font (size 1.27 1.27)) hide)
+    )
+    (property "Datasheet" "~" (id 3) (at 44.45 31.75 0)
+      (effects (font (size 1.27 1.27)) hide)
+    )
+  )
   (symbol (lib_id "power:GND") (at 209.55 67.31 270) (unit 1)
     (in_bom yes) (on_board yes)
@@
     (pin "1")
   )
+  (symbol (lib_id "Mechanical:MountingHole") (at 238.76 132.08 0) (unit 1)
+    (in_bom yes) (on_board yes)
+    (property "Reference" "H3" (id 0) (at 241.3 130.9116 0)
+      (effects (font (size 1.27 1.27)) (justify left))
+    )
+    (property "Value" "MountingHole" (id 1) (at 241.3 133.223 0)
+      (effects (font (size 1.27 1.27)) (justify left))
+    )
+    (property "Footprint" "MountingHole:MountingHole_3.2mm_M3_ISO7380_Pad" (id 2) (at 238.76 132.08 0)
+      (effects (font (size 1.27 1.27)) hide)
+    )
+    (property "Datasheet" "~" (id 3) (at 238.76 132.08 0)
+      (effects (font (size 1.27 1.27)) hide)
+    )
+  )
   (symbol (lib_id "power:VCC") (at 209.55 64.77 90) (unit 1)
     (in_bom yes) (on_board yes)
@@
     )
     (pin "1")
+  )
+  (symbol (lib_id "Mechanical:MountingHole") (at 242.57 35.56 0) (unit 1)
+    (in_bom yes) (on_board yes)
+    (property "Reference" "H4" (id 0) (at 245.11 34.3916 0)
+      (effects (font (size 1.27 1.27)) (justify left))
+    )
+    (property "Value" "MountingHole" (id 1) (at 245.11 36.703 0)
+      (effects (font (size 1.27 1.27)) (justify left))
+    )
+    (property "Footprint" "MountingHole:MountingHole_3.2mm_M3_ISO7380_Pad" (id 2) (at 242.57 35.56 0)
+      (effects (font (size 1.27 1.27)) hide)
+    )
+    (property "Datasheet" "~" (id 3) (at 242.57 35.56 0)
+      (effects (font (size 1.27 1.27)) hide)
+    )
   )
   (symbol (lib_id "power:VEE") (at 209.55 69.85 90) (unit 1)
@@
       (reference "F3") (unit 1) (value "F0.2A") (footprint "Fuse:Fuseholder_Clip-5x20mm_Littelfuse_111_Inline_P20.00x5.00mm_D1.05mm_Horizontal")
     )
-    (path "/259bb928-7a55-4782-aba9-7b00086dca40/82fd8dbd-f40b-4d34-be16-2dcfee874c86"
+    (path "/13582fea-ab85-4aaf-98b0-481a365923da"
       (reference "H1") (unit 1) (value "MountingHole") (footprint "MountingHole:MountingHole_3.2mm_M3_ISO7380_Pad")
     )
-    (path "/259bb928-7a55-4782-aba9-7b00086dca40/72e5286a-630f-4e9d-8734-127a0eac58da"
+    (path "/718736b5-41f2-4b9f-925a-c9407d26c72e"
       (reference "H2") (unit 1) (value "MountingHole") (footprint "MountingHole:MountingHole_3.2mm_M3_ISO7380_Pad")
     )
-    (path "/259bb928-7a55-4782-aba9-7b00086dca40/d821fe4b-53ed-454f-8da8-80ab350f69ef"
+    (path "/a4da4b46-ced5-4889-9646-403ca62ec0e2"
       (reference "H3") (unit 1) (value "MountingHole") (footprint "MountingHole:MountingHole_3.2mm_M3_ISO7380_Pad")
     )
-    (path "/259bb928-7a55-4782-aba9-7b00086dca40/0644f46e-d29c-47b3-8639-ef08b882c5fe"
+    (path "/fc7cbf6d-41ae-48e4-9f41-d633c5fd5f6e"
       (reference "H4") (unit 1) (value "MountingHole") (footprint "MountingHole:MountingHole_3.2mm_M3_ISO7380_Pad")
     )
